Commit message: Remove stuff related to unused parameter kinematics_file

File: rbkairos_description/robots/versions/rbkairos_ur10_wsg50.urdf.xacro (robot description, xacro)
@@ -16,12 +16,11 @@
 	<xacro:arg name="ros_planar_move_plugin" default="false"/>
 	<xacro:arg name="has_arm" default="true"/>
-    <xacro:arg name="load_kinematics_file" default="false"/> <!-- Necesarry for ur_description compatible with official ur drivers-->
-    <xacro:property name="arm_position_x" value="0.0"/>
-    <xacro:property name="arm_position_y" value="0"/>
-    <xacro:property name="arm_position_z" value="0.383612"/>
-    <xacro:property name="arm_orientation_r" value="0"/>
-    <xacro:property name="arm_orientation_p" value="0"/>
-    <xacro:property name="arm_orientation_y" value="0"/>
-  <xacro:macro name="rbkairos" params="prefix publish_bf hq load_kinematics_file">
+	<xacro:property name="arm_position_x" value="0.0"/>
+	<xacro:property name="arm_position_y" value="0"/>
+	<xacro:property name="arm_position_z" value="0.383612"/>
+	<xacro:property name="arm_orientation_r" value="0"/>
+	<xacro:property name="arm_orientation_p" value="0"/>
+	<xacro:property name="arm_orientation_y" value="0"/>
+  <xacro:macro name="rbkairos" params="prefix publish_bf hq">
 		<!-- *************** -->
 		<!-- Robots Elements -->
@@ -30,28 +29,14 @@
 		<!-- RBKAIROS base -->
 		<xacro:rbkairos_base prefix="$(arg prefix)" publish_bf="true" hq="true"/>
-        <!-- UR-10 ARM -->
-		<xacro:if value="$(arg load_kinematics_file)">
-			<xacro:ur10_robot prefix="$(arg prefix)arm_" joint_limited="true"
-			shoulder_pan_lower_limit="${-pi}" shoulder_pan_upper_limit="${pi}"
-			wrist_3_lower_limit="${-pi}" wrist_3_upper_limit="${pi}"
-			kinematics_file="${load_yaml('$(find rbkairos_control)/config/ur10_calibration.yaml')}">
-			</xacro:ur10_robot>
-			<joint name="$(arg prefix)arm_base_joint" type="fixed">
-				<origin xyz="${arm_position_x} ${arm_position_y} ${arm_position_z}" rpy="${arm_orientation_r} ${arm_orientation_p} ${arm_orientation_y}"/>
-				<parent link="$(arg prefix)base_link" />
-				<child link="$(arg prefix)arm_base_link" />
-			</joint>
-		</xacro:if>
-		<xacro:unless value="$(arg load_kinematics_file)">
-			<xacro:ur10_robot prefix="$(arg prefix)arm_" joint_limited="true"
-			shoulder_pan_lower_limit="${-pi}" shoulder_pan_upper_limit="${pi}"
-			wrist_3_lower_limit="${-pi}" wrist_3_upper_limit="${pi}">
-			</xacro:ur10_robot>
-			<joint name="$(arg prefix)arm_base_joint" type="fixed">
+    <!-- UR-10 ARM -->
+		<xacro:ur10_robot prefix="$(arg prefix)arm_" joint_limited="true"
+		shoulder_pan_lower_limit="${-pi}" shoulder_pan_upper_limit="${pi}"
+		wrist_3_lower_limit="${-pi}" wrist_3_upper_limit="${pi}">
+		</xacro:ur10_robot>
+		<joint name="$(arg prefix)arm_base_joint" type="fixed">
 			<origin xyz="${arm_position_x} ${arm_position_y} ${arm_position_z}" rpy="${arm_orientation_r} ${arm_orientation_p} ${arm_orientation_y}"/>
 			<parent link="$(arg prefix)base_link" />
 			<child link="$(arg prefix)arm_base_link" />
-			</joint>
-		</xacro:unless>
+		</joint>
 		<!-- Schunk WSG-50 -->
 		<xacro:wsg_50_xacro name="$(arg prefix)wsg50" parent="$(arg prefix)arm_tool0" finger_length="0.023" finger_tip="0">
@@ -64,4 +49,4 @@
 	   <xacro:omni_steering prefix="$(arg prefix)" publish_tf="true"/>
    </xacro:if>
-   <xacro:rbkairos prefix="$(arg prefix)" publish_bf="true" hq="true" load_kinematics_file="$(arg load_kinematics_file)"/>
+   <xacro:rbkairos prefix="$(arg prefix)" publish_bf="true" hq="true"/>
 </robot>
